Commit message: add estimator

File: src/asserts/aliengo/aliengo.urdf (robot description, URDF)
Before this commit: robot aliengo_description, 18 links, 17 joints
Links:
- removed link FL_foot
- removed link FR_foot
- removed link RL_foot
- removed link RR_foot
- added link fl_foot, mass 0.06; collision sphere radius=0.0265; visual sphere radius=0.0165
- added link fr_foot, mass 0.06; collision sphere radius=0.0265; visual sphere radius=0.0165
- added link rl_foot, mass 0.06; collision sphere radius=0.0265; visual sphere radius=0.0165
- added link rr_foot, mass 0.06; collision sphere radius=0.0265; visual sphere radius=0.0165
Joints:
- joint FL_foot_fixed: child FL_foot -> fl_foot
- joint FR_foot_fixed: child FR_foot -> fr_foot
- joint RL_foot_fixed: child RL_foot -> rl_foot
- joint RR_foot_fixed: child RR_foot -> rr_foot

Commit message: reorder

File: src/asserts/aliengo/aliengo.urdf (robot description, URDF)
Before this commit: robot aliengo_description, 18 links, 17 joints
Links:
- link FL_calf: geometry collision box size=0.25 0.0208 0.016; visual mesh filename=package://asserts/aliengo/meshes/calf.stl scale=1 1 1
- link FL_hip: geometry collision cylinder length=0.0418 radius=0.046; visual mesh filename=package://asserts/aliengo/meshes/hip.stl scale=1 1 1
- link FL_thigh: geometry collision box size=0.25 0.0374 0.043; visual mesh filename=package://asserts/aliengo/meshes/thigh.stl scale=1 1 1
- link FR_calf: geometry collision box size=0.25 0.0208 0.016; visual mesh filename=package://asserts/aliengo/meshes/calf.stl scale=1 1 1
- link FR_hip: geometry collision cylinder length=0.0418 radius=0.046; visual mesh filename=package://asserts/aliengo/meshes/hip.stl scale=1 1 1
- link FR_thigh: geometry collision box size=0.25 0.0374 0.043; visual mesh filename=package://asserts/aliengo/meshes/thigh_mirror.stl scale=1 1 1
- link RL_calf: geometry collision box size=0.25 0.0208 0.016; visual mesh filename=package://asserts/aliengo/meshes/calf.stl scale=1 1 1
- link RL_hip: geometry collision cylinder length=0.0418 radius=0.046; visual mesh filename=package://asserts/aliengo/meshes/hip.stl scale=1 1 1
- link RL_thigh: geometry collision box size=0.25 0.0374 0.043; visual mesh filename=package://asserts/aliengo/meshes/thigh.stl scale=1 1 1
- link RR_calf: geometry collision box size=0.25 0.0208 0.016; visual mesh filename=package://asserts/aliengo/meshes/calf.stl scale=1 1 1
- link RR_hip: geometry collision cylinder length=0.0418 radius=0.046; visual mesh filename=package://asserts/aliengo/meshes/hip.stl scale=1 1 1
- link RR_thigh: geometry collision box size=0.25 0.0374 0.043; visual mesh filename=package://asserts/aliengo/meshes/thigh_mirror.stl scale=1 1 1
- link trunk: geometry collision box size=0.647 0.15 0.112; visual mesh filename=package://asserts/aliengo/meshes/trunk.stl scale=1 1 1
