Commit message: update

File: src/asserts/a1/a1.urdf (robot description, URDF)
Before this commit: robot a1, 18 links, 17 joints
Links:
- added link FL_thigh_shoulder; collision cylinder length=0.032 radius=0.041
- added link FR_thigh_shoulder; collision cylinder length=0.032 radius=0.041
- added link RL_thigh_shoulder; collision cylinder length=0.032 radius=0.041
- added link RR_thigh_shoulder; collision cylinder length=0.032 radius=0.041
- link FL_hip: geometry collision cylinder length=0.04 radius=0.046; visual mesh filename=package://asserts/a1/meshes/hip.stl scale=1 1 1
- link FR_hip: geometry collision cylinder length=0.04 radius=0.046; visual mesh filename=package://asserts/a1/meshes/hip.stl scale=1 1 1
- link RL_hip: geometry collision cylinder length=0.04 radius=0.046; visual mesh filename=package://asserts/a1/meshes/hip.stl scale=1 1 1
- link RR_hip: geometry collision cylinder length=0.04 radius=0.046; visual mesh filename=package://asserts/a1/meshes/hip.stl scale=1 1 1
- link trunk: mass 4.713 -> 6.0
Joints:
- added joint FL_hip_fixed: type fixed, parent FL_hip, child FL_thigh_shoulder, origin xyz=0 0.081 0 rpy=0 0 0
- added joint FR_hip_fixed: type fixed, parent FR_hip, child FR_thigh_shoulder, origin xyz=0 -0.081 0 rpy=0 0 0
- added joint RL_hip_fixed: type fixed, parent RL_hip, child RL_thigh_shoulder, origin xyz=0 0.081 0 rpy=0 0 0
- added joint RR_hip_fixed: type fixed, parent RR_hip, child RR_thigh_shoulder, origin xyz=0 -0.081 0 rpy=0 0 0
- joint FL_calf_joint: limit lower=-2.69653369433 upper=-0.916297857297 effort=55 velocity=28.6 -> lower=-2.69653369433 upper=-0.916297857297 effort=33.5 velocity=21
- joint FL_hip_joint: limit lower=-0.802851455917 upper=0.802851455917 effort=20 velocity=52.4 -> lower=-0.802851455917 upper=0.802851455917 effort=33.5 velocity=21; origin xyz=0.183 0.047 0 rpy=0 0 0 -> xyz=0.1805 0.047 0 rpy=0 0 0
- joint FL_thigh_joint: limit lower=-1.0471975512 upper=4.18879020479 effort=55 velocity=28.6 -> lower=-1.0471975512 upper=4.18879020479 effort=33.5 velocity=21; origin xyz=0 0.08505 0 rpy=0 0 0 -> xyz=0 0.0838 0 rpy=0 0 0
- joint FR_calf_joint: limit lower=-2.69653369433 upper=-0.916297857297 effort=55 velocity=28.6 -> lower=-2.69653369433 upper=-0.916297857297 effort=33.5 velocity=21
- joint FR_hip_joint: limit lower=-0.802851455917 upper=0.802851455917 effort=20 velocity=52.4 -> lower=-0.802851455917 upper=0.802851455917 effort=33.5 velocity=21; origin xyz=0.183 -0.047 0 rpy=0 0 0 -> xyz=0.1805 -0.047 0 rpy=0 0 0
- joint FR_thigh_joint: limit lower=-1.0471975512 upper=4.18879020479 effort=55 velocity=28.6 -> lower=-1.0471975512 upper=4.18879020479 effort=33.5 velocity=21; origin xyz=0 -0.08505 0 rpy=0 0 0 -> xyz=0 -0.0838 0 rpy=0 0 0
- joint RL_calf_joint: limit lower=-2.69653369433 upper=-0.916297857297 effort=55 velocity=28.6 -> lower=-2.69653369433 upper=-0.916297857297 effort=33.5 velocity=21
- joint RL_hip_joint: limit lower=-0.802851455917 upper=0.802851455917 effort=20 velocity=52.4 -> lower=-0.802851455917 upper=0.802851455917 effort=33.5 velocity=21; origin xyz=-0.183 0.047 0 rpy=0 0 0 -> xyz=-0.1805 0.047 0 rpy=0 0 0
- joint RL_thigh_joint: limit lower=-1.0471975512 upper=4.18879020479 effort=55 velocity=28.6 -> lower=-1.0471975512 upper=4.18879020479 effort=33.5 velocity=21; origin xyz=0 0.08505 0 rpy=0 0 0 -> xyz=0 0.0838 0 rpy=0 0 0
- joint RR_calf_joint: limit lower=-2.69653369433 upper=-0.916297857297 effort=55 velocity=28.6 -> lower=-2.69653369433 upper=-0.916297857297 effort=33.5 velocity=21
- joint RR_hip_joint: limit lower=-0.802851455917 upper=0.802851455917 effort=20 velocity=52.4 -> lower=-0.802851455917 upper=0.802851455917 effort=33.5 velocity=21; origin xyz=-0.183 -0.047 0 rpy=0 0 0 -> xyz=-0.1805 -0.047 0 rpy=0 0 0
- joint RR_thigh_joint: limit lower=-1.0471975512 upper=4.18879020479 effort=55 velocity=28.6 -> lower=-1.0471975512 upper=4.18879020479 effort=33.5 velocity=21; origin xyz=0 -0.08505 0 rpy=0 0 0 -> xyz=0 -0.0838 0 rpy=0 0 0

Commit message: roll back

File: src/asserts/a1/a1.urdf (robot description, URDF)
Before this commit: robot a1, 22 links, 21 joints
Links:
- removed link FL_thigh_shoulder
- removed link FR_thigh_shoulder
- removed link RL_thigh_shoulder
- removed link RR_thigh_shoulder
- link FL_hip: geometry collision cylinder length=0.08 radius=0.04; visual mesh filename=package://asserts/a1/meshes/hip.stl scale=1 1 1
- link FR_hip: geometry collision cylinder length=0.08 radius=0.04; visual mesh filename=package://asserts/a1/meshes/hip.stl scale=1 1 1
- link RL_hip: geometry collision cylinder length=0.08 radius=0.04; visual mesh filename=package://asserts/a1/meshes/hip.stl scale=1 1 1
- link RR_hip: geometry collision cylinder length=0.08 radius=0.04; visual mesh filename=package://asserts/a1/meshes/hip.stl scale=1 1 1
- link trunk: mass 6.0 -> 4.713
Joints:
- removed joint FL_hip_fixed
- removed joint FR_hip_fixed
- removed joint RL_hip_fixed
- removed joint RR_hip_fixed
- joint FL_calf_joint: limit lower=-2.69653369433 upper=-0.916297857297 effort=33.5 velocity=21 -> lower=-2.69653369433 upper=-0.916297857297 effort=55 velocity=28.6
- joint FL_hip_joint: limit lower=-0.802851455917 upper=0.802851455917 effort=33.5 velocity=21 -> lower=-0.802851455917 upper=0.802851455917 effort=20 velocity=52.4; origin xyz=0.1805 0.047 0 rpy=0 0 0 -> xyz=0.183 0.047 0 rpy=0 0 0
- joint FL_thigh_joint: limit lower=-1.0471975512 upper=4.18879020479 effort=33.5 velocity=21 -> lower=-1.0471975512 upper=4.18879020479 effort=55 velocity=28.6; origin xyz=0 0.0838 0 rpy=0 0 0 -> xyz=0 0.08505 0 rpy=0 0 0
- joint FR_calf_joint: limit lower=-2.69653369433 upper=-0.916297857297 effort=33.5 velocity=21 -> lower=-2.69653369433 upper=-0.916297857297 effort=55 velocity=28.6
- joint FR_hip_joint: limit lower=-0.802851455917 upper=0.802851455917 effort=33.5 velocity=21 -> lower=-0.802851455917 upper=0.802851455917 effort=20 velocity=52.4; origin xyz=0.1805 -0.047 0 rpy=0 0 0 -> xyz=0.183 -0.047 0 rpy=0 0 0
- joint FR_thigh_joint: limit lower=-1.0471975512 upper=4.18879020479 effort=33.5 velocity=21 -> lower=-1.0471975512 upper=4.18879020479 effort=55 velocity=28.6; origin xyz=0 -0.0838 0 rpy=0 0 0 -> xyz=0 -0.08505 0 rpy=0 0 0
- joint RL_calf_joint: limit lower=-2.69653369433 upper=-0.916297857297 effort=33.5 velocity=21 -> lower=-2.69653369433 upper=-0.916297857297 effort=55 velocity=28.6
- joint RL_hip_joint: limit lower=-0.802851455917 upper=0.802851455917 effort=33.5 velocity=21 -> lower=-0.802851455917 upper=0.802851455917 effort=20 velocity=52.4; origin xyz=-0.1805 0.047 0 rpy=0 0 0 -> xyz=-0.183 0.047 0 rpy=0 0 0
- joint RL_thigh_joint: limit lower=-1.0471975512 upper=4.18879020479 effort=33.5 velocity=21 -> lower=-1.0471975512 upper=4.18879020479 effort=55 velocity=28.6; origin xyz=0 0.0838 0 rpy=0 0 0 -> xyz=0 0.08505 0 rpy=0 0 0
- joint RR_calf_joint: limit lower=-2.69653369433 upper=-0.916297857297 effort=33.5 velocity=21 -> lower=-2.69653369433 upper=-0.916297857297 effort=55 velocity=28.6
- joint RR_hip_joint: limit lower=-0.802851455917 upper=0.802851455917 effort=33.5 velocity=21 -> lower=-0.802851455917 upper=0.802851455917 effort=20 velocity=52.4; origin xyz=-0.1805 -0.047 0 rpy=0 0 0 -> xyz=-0.183 -0.047 0 rpy=0 0 0
- joint RR_thigh_joint: limit lower=-1.0471975512 upper=4.18879020479 effort=33.5 velocity=21 -> lower=-1.0471975512 upper=4.18879020479 effort=55 velocity=28.6; origin xyz=0 -0.0838 0 rpy=0 0 0 -> xyz=0 -0.08505 0 rpy=0 0 0

Commit message: update better the last one

File: src/asserts/a1/a1.urdf (robot description, URDF)
Before this commit: robot a1, 22 links, 21 joints
Links:
- removed link FL_thigh_shoulder
- removed link FR_thigh_shoulder
- removed link RL_thigh_shoulder
- removed link RR_thigh_shoulder
- link FL_hip: geometry collision cylinder length=0.08 radius=0.04; visual mesh filename=package://asserts/a1/meshes/hip.stl scale=1 1 1
- link FR_hip: geometry collision cylinder length=0.08 radius=0.04; visual mesh filename=package://asserts/a1/meshes/hip.stl scale=1 1 1
- link RL_hip: geometry collision cylinder length=0.08 radius=0.04; visual mesh filename=package://asserts/a1/meshes/hip.stl scale=1 1 1
- link RR_hip: geometry collision cylinder length=0.08 radius=0.04; visual mesh filename=package://asserts/a1/meshes/hip.stl scale=1 1 1
- link trunk: mass 6.0 -> 5.713
Joints:
- removed joint FL_hip_fixed
- removed joint FR_hip_fixed
- removed joint RL_hip_fixed
- removed joint RR_hip_fixed
- joint FL_calf_joint: limit lower=-2.69653369433 upper=-0.916297857297 effort=33.5 velocity=21 -> lower=-2.69653369433 upper=-0.916297857297 effort=55 velocity=28.6
- joint FL_hip_joint: limit lower=-0.802851455917 upper=0.802851455917 effort=33.5 velocity=21 -> lower=-0.802851455917 upper=0.802851455917 effort=20 velocity=52.4; origin xyz=0.1805 0.047 0 rpy=0 0 0 -> xyz=0.183 0.047 0 rpy=0 0 0
- joint FL_thigh_joint: limit lower=-1.0471975512 upper=4.18879020479 effort=33.5 velocity=21 -> lower=-1.0471975512 upper=4.18879020479 effort=55 velocity=28.6; origin xyz=0 0.0838 0 rpy=0 0 0 -> xyz=0 0.08505 0 rpy=0 0 0
- joint FR_calf_joint: limit lower=-2.69653369433 upper=-0.916297857297 effort=33.5 velocity=21 -> lower=-2.69653369433 upper=-0.916297857297 effort=55 velocity=28.6
- joint FR_hip_joint: limit lower=-0.802851455917 upper=0.802851455917 effort=33.5 velocity=21 -> lower=-0.802851455917 upper=0.802851455917 effort=20 velocity=52.4; origin xyz=0.1805 -0.047 0 rpy=0 0 0 -> xyz=0.183 -0.047 0 rpy=0 0 0
- joint FR_thigh_joint: limit lower=-1.0471975512 upper=4.18879020479 effort=33.5 velocity=21 -> lower=-1.0471975512 upper=4.18879020479 effort=55 velocity=28.6; origin xyz=0 -0.0838 0 rpy=0 0 0 -> xyz=0 -0.08505 0 rpy=0 0 0
- joint RL_calf_joint: limit lower=-2.69653369433 upper=-0.916297857297 effort=33.5 velocity=21 -> lower=-2.69653369433 upper=-0.916297857297 effort=55 velocity=28.6
- joint RL_hip_joint: limit lower=-0.802851455917 upper=0.802851455917 effort=33.5 velocity=21 -> lower=-0.802851455917 upper=0.802851455917 effort=20 velocity=52.4; origin xyz=-0.1805 0.047 0 rpy=0 0 0 -> xyz=-0.183 0.047 0 rpy=0 0 0
- joint RL_thigh_joint: limit lower=-1.0471975512 upper=4.18879020479 effort=33.5 velocity=21 -> lower=-1.0471975512 upper=4.18879020479 effort=55 velocity=28.6; origin xyz=0 0.0838 0 rpy=0 0 0 -> xyz=0 0.08505 0 rpy=0 0 0
- joint RR_calf_joint: limit lower=-2.69653369433 upper=-0.916297857297 effort=33.5 velocity=21 -> lower=-2.69653369433 upper=-0.916297857297 effort=55 velocity=28.6
- joint RR_hip_joint: limit lower=-0.802851455917 upper=0.802851455917 effort=33.5 velocity=21 -> lower=-0.802851455917 upper=0.802851455917 effort=20 velocity=52.4; origin xyz=-0.1805 -0.047 0 rpy=0 0 0 -> xyz=-0.183 -0.047 0 rpy=0 0 0
- joint RR_thigh_joint: limit lower=-1.0471975512 upper=4.18879020479 effort=33.5 velocity=21 -> lower=-1.0471975512 upper=4.18879020479 effort=55 velocity=28.6; origin xyz=0 -0.0838 0 rpy=0 0 0 -> xyz=0 -0.08505 0 rpy=0 0 0

Commit message: good for experiments ( proposed method v.s. user-tuned  + MPC)

File: src/asserts/a1/a1.urdf (robot description, URDF)
Before this commit: robot a1, 18 links, 17 joints
Links:
- link trunk: mass 5.713 -> 4.713
