Commit message: update

File: src/asserts/p1/PF_A.urdf (robot description, URDF)
Before this commit: robot PF_A, 11 links, 10 joints
Links:
- link abad_L: geometry collision mesh filename=package://asserts/p1/meshes/abad_L_Link.STL; visual mesh filename=package://asserts/p1/meshes/abad_L_Link.STL
- link abad_R: geometry collision mesh filename=package://asserts/p1/meshes/abad_R_Link.STL; visual mesh filename=package://asserts/p1/meshes/abad_R_Link.STL
- link base: geometry collision mesh filename=package://asserts/p1/meshes/base_Link.STL; visual mesh filename=package://asserts/p1/meshes/base_Link.STL
- link foot_L: geometry collision mesh filename=package://asserts/p1/meshes/foot_L_Link.STL; visual mesh filename=package://asserts/p1/meshes/foot_L_Link.STL
- link foot_R: geometry collision mesh filename=package://asserts/p1/meshes/foot_R_Link.STL; visual mesh filename=package://asserts/p1/meshes/foot_R_Link.STL
- link hip_L: geometry collision mesh filename=package://asserts/p1/meshes/hip_L_Link.STL; visual mesh filename=package://asserts/p1/meshes/hip_L_Link.STL
- link hip_R: geometry collision mesh filename=package://asserts/p1/meshes/hip_R_Link.STL; visual mesh filename=package://asserts/p1/meshes/hip_R_Link.STL
- link knee_L: geometry collision mesh filename=package://asserts/p1/meshes/knee_L_Link.STL; visual mesh filename=package://asserts/p1/meshes/knee_L_Link.STL
- link knee_R: geometry collision mesh filename=package://asserts/p1/meshes/knee_R_Link.STL; visual mesh filename=package://asserts/p1/meshes/knee_R_Link.STL

Commit message: update

File: src/asserts/p1/PF_A.urdf (robot description, URDF)
Before this commit: robot PF_A, 11 links, 10 joints
Links:
- removed link abad_L
- removed link abad_R
- removed link foot_L
- removed link foot_R
- removed link hip_L
- removed link hip_R
- removed link knee_L
- removed link knee_R
- removed link limx_imu
- removed link world
- added link abad_L_Link, mass 1.03648983; collision cylinder length=0.15 radius=0.05; visual mesh filename=package://asserts/p1/meshes/abad_left_link.STL
- added link abad_R_Link, mass 1.03648872; collision cylinder length=0.15 radius=0.05; visual mesh filename=package://asserts/p1/meshes/abad_right_link.STL
- added link foot_L_Link, mass 0.14047647; collision sphere radius=0.035; visual mesh filename=package://asserts/p1/meshes/foot_left_link.STL
- added link foot_R_Link, mass 0.14047647; collision sphere radius=0.035; visual mesh filename=package://asserts/p1/meshes/foot_right_link.STL
- added link hip_L_Link, mass 1.73405445; collision cylinder length=0.22 radius=0.035; visual mesh filename=package://asserts/p1/meshes/hip_left_link.STL
- added link hip_R_Link, mass 1.73405240; collision cylinder length=0.22 radius=0.035; visual mesh filename=package://asserts/p1/meshes/hip_right_link.STL
- added link knee_L_Link, mass 0.25930748; collision cylinder length=0.26 radius=0.015; visual mesh filename=package://asserts/p1/meshes/knee_left_link.STL
- added link knee_R_Link, mass 0.25930895; collision cylinder length=0.26 radius=0.015; visual mesh filename=package://asserts/p1/meshes/knee_right_link.STL
- link base: geometry collision box size=0.2 0.3 0.15; visual mesh filename=package://asserts/p1/meshes/base_link.STL
Joints:
- removed joint abad_L_joint
- removed joint abad_R_joint
- removed joint fixed
- removed joint foot_L_joint
- removed joint foot_R_joint
- removed joint hip_L_joint
- removed joint hip_R_joint
- removed joint knee_L_joint
- removed joint knee_R_joint
- removed joint limx_imu_joint
- added joint abad_L_Joint: type revolute, parent base, child abad_L_Link, origin xyz=0.0142 0.095 -0.08176 rpy=0 0 0, axis 1 0 0, limit lower=-0.383972435 upper=0.785398163 effort=40.0 velocity=15.0
- added joint abad_R_Joint: type revolute, parent base, child abad_R_Link, origin xyz=0.0142 -0.095 -0.08176 rpy=0 0 0, axis 1 0 0, limit lower=-0.785398163 upper=0.383972435 effort=40.0 velocity=15.0
- added joint foot_L_Joint: type fixed, parent knee_L_Link, child foot_L_Link, origin xyz=0.15 0 -0.29066 rpy=0 0 0, axis 0 0 0
- added joint foot_R_Joint: type fixed, parent knee_R_Link, child foot_R_Link, origin xyz=0.15 0 -0.29066 rpy=0 0 0, axis 0 0 0
- added joint hip_L_Joint: type revolute, parent abad_L_Link, child hip_L_Link, origin xyz=-0.0802 0.031 0 rpy=0 0 0, axis 0 1 0, limit lower=-1.047197551 upper=1.483529864 effort=40.0 velocity=15.0
- added joint hip_R_Joint: type revolute, parent abad_R_Link, child hip_R_Link, origin xyz=-0.0802 -0.031 0 rpy=0 0 0, axis 0 -1 0, limit lower=-1.483529864 upper=1.047197551 effort=40.0 velocity=15.0
- added joint knee_L_Joint: type revolute, parent hip_L_Link, child knee_L_Link, origin xyz=-0.15 -0.021 -0.25981 rpy=0 0 0, axis 0 -1 0, limit lower=-1.012290966 upper=1.256637061 effort=40 velocity=15.0
- added joint knee_R_Joint: type revolute, parent hip_R_Link, child knee_R_Link, origin xyz=-0.15 0.021 -0.25981 rpy=0 0 0, axis 0 1 0, limit lower=-1.256637061 upper=1.012290966 effort=40.0 velocity=15.0
